Commit message: Sync changes

File: src/RobotSimulator/src/robot_sim/urdf/markers.xacro (robot description, xacro)
@@ -5,9 +5,9 @@
   <!-- Base link -->
   <link name="world"/>
-  <joint name="target_joint" type="fixed">
+  <joint name="marker_red_joint" type="fixed">
     <parent link="world"/>
-    <child link="target"/>
+    <child link="marker_red"/>
   </joint>
-  <link name="target">
+  <link name="marker_red">
     <visual>
       <origin xyz="0 0 0" rpy="0 0 0"/>
@@ -26,5 +26,5 @@
     </inertial>
   </link>
-  <gazebo reference="target">
+  <gazebo reference="marker_red">
     <material>Gazebo/Red</material>
   </gazebo>

Commit message: A star (incomplete)

File: src/RobotSimulator/src/robot_sim/urdf/markers.xacro (robot description, xacro)
@@ -10,4 +10,10 @@
   </joint>
   <link name="marker_red">
+    <collision>
+      <origin xyz="0 0 0" rpy="0 0 0"/>
+      <geometry>
+	      <sphere radius="${marker_point_radius}" />
+      </geometry>
+    </collision>
     <visual>
       <origin xyz="0 0 0" rpy="0 0 0"/>

File: src/RobotSimulator/src/robot_sim/urdf/robot.xacro (robot description, xacro)
@@ -30,6 +30,6 @@
   <xacro:property name="joint2_low" value="-1.529065" />
   <xacro:property name="joint2_high" value="1.571069" />
-  <xacro:property name="joint3_low" value="-1.570796" />
-  <xacro:property name="joint3_high" value="1.570796" />
+  <xacro:property name="joint3_low" value="-0.785398" />
+  <xacro:property name="joint3_high" value="0.785398" />
   <xacro:property name="joint4_low" value="-3.053450" />
   <xacro:property name="joint4_high" value="3.053439" />

Commit message: Implement A* + artificial potential field

File: src/RobotSimulator/src/robot_sim/urdf/markers.xacro (robot description, xacro)
@@ -10,10 +10,4 @@
   </joint>
   <link name="marker_red">
-    <collision>
-      <origin xyz="0 0 0" rpy="0 0 0"/>
-      <geometry>
-	      <sphere radius="${marker_point_radius}" />
-      </geometry>
-    </collision>
     <visual>
       <origin xyz="0 0 0" rpy="0 0 0"/>

File: src/RobotSimulator/src/robot_sim/urdf/obstacles.xacro (robot description, xacro)
@@ -9,5 +9,5 @@
     <parent link="world"/>
     <child link="table"/>
-    <origin xyz="0 0 0.5" rpy="0 0 0"/>
+    <origin xyz="0 0 0.1" rpy="0 0 0"/>
   </joint>
   <link name="table">
@@ -15,5 +15,5 @@
       <origin xyz="0 0 0" rpy="0 0 0"/>
       <geometry>
-	      <box size="1 1 1" />
+	      <box size="1 1 0.2" />
       </geometry>
     </collision>
@@ -21,5 +21,5 @@
       <origin xyz="0 0 0" rpy="0 0 0"/>
       <geometry>
-	      <box size="1 1 1" />
+	      <box size="1 1 0.2" />
       </geometry>
       <material name="white"/>
@@ -41,8 +41,9 @@
     <parent link="world"/>
     <child link="obj1"/>
+    <origin xyz="0.701 0.701 2" rpy="0 0 0"/>
   </joint>
   <link name="obj1">
     <collision>
-      <origin xyz="0.701 0.701 2" rpy="0 0 0"/>
+      <origin xyz="0 0 0" rpy="0 0 0"/>
       <geometry>
 	      <box size="0.302 0.302 4"/>
@@ -50,5 +51,5 @@
     </collision>
     <visual>
-      <origin xyz="0.701 0.701 2" rpy="0 0 0"/>
+      <origin xyz="0 0 0" rpy="0 0 0"/>
       <geometry>
 	      <box size="0.302 0.302 4"/>
@@ -57,5 +58,5 @@
     </visual>
     <inertial>
-      <origin xyz="0.701 0.701 2" rpy="0 0 0"/>
+      <origin xyz="0 0 0" rpy="0 0 0"/>
       <mass value="1.0"/>
       <inertia
@@ -72,8 +73,9 @@
     <parent link="world"/>
     <child link="obj2"/>
+    <origin xyz="0.701 -0.701 2" rpy="0 0 0"/>
   </joint>
   <link name="obj2">
     <collision>
-      <origin xyz="0.701 -0.701 2" rpy="0 0 0"/>
+      <origin xyz="0 0 0" rpy="0 0 0"/>
       <geometry>
 	      <box size="0.302 0.302 4"/>
@@ -81,5 +83,5 @@
     </collision>
     <visual>
-      <origin xyz="0.701 -0.701 2" rpy="0 0 0"/>
+      <origin xyz="0 0 0" rpy="0 0 0"/>
       <geometry>
 	      <box size="0.302 0.302 4"/>
@@ -88,5 +90,5 @@
     </visual>
     <inertial>
-      <origin xyz="0.701 -0.701 2" rpy="0 0 0"/>
+      <origin xyz="0 0 0" rpy="0 0 0"/>
       <mass value="1.0"/>
       <inertia
@@ -103,8 +105,9 @@
     <parent link="world"/>
     <child link="obj3"/>
+    <origin xyz="-0.701 0.701 2" rpy="0 0 0"/>
   </joint>
   <link name="obj3">
     <collision>
-      <origin xyz="-0.701 0.701 2" rpy="0 0 0"/>
+      <origin xyz="0 0 0" rpy="0 0 0"/>
       <geometry>
 	      <box size="0.302 0.302 4"/>
@@ -112,5 +115,5 @@
     </collision>
     <visual>
-      <origin xyz="-0.701 0.701 2" rpy="0 0 0"/>
+      <origin xyz="0 0 0" rpy="0 0 0"/>
       <geometry>
 	      <box size="0.302 0.302 4"/>
@@ -119,5 +122,5 @@
     </visual>
     <inertial>
-      <origin xyz="-0.701 0.701 2" rpy="0 0 0"/>
+      <origin xyz="0 0 0" rpy="0 0 0"/>
       <mass value="1.0"/>
       <inertia
@@ -134,8 +137,9 @@
     <parent link="world"/>
     <child link="obj4"/>
+    <origin xyz="-0.701 -0.701 2" rpy="0 0 0"/>
   </joint>
   <link name="obj4">
     <collision>
-      <origin xyz="-0.701 -0.701 2" rpy="0 0 0"/>
+      <origin xyz="0 0 0" rpy="0 0 0"/>
       <geometry>
 	      <box size="0.302 0.302 4"/>
@@ -143,5 +147,5 @@
     </collision>
     <visual>
-      <origin xyz="-0.701 -0.701 2" rpy="0 0 0"/>
+      <origin xyz="0 0 0" rpy="0 0 0"/>
       <geometry>
 	      <box size="0.302 0.302 4"/>
@@ -150,5 +154,5 @@
     </visual>
     <inertial>
-      <origin xyz="-0.701 -0.701 2" rpy="0 0 0"/>
+      <origin xyz="0 0 0" rpy="0 0 0"/>
       <mass value="1.0"/>
       <inertia

File: src/RobotSimulator/src/robot_sim/urdf/robot.xacro (robot description, xacro)
@@ -21,4 +21,5 @@
   <xacro:property name="link3_length" value="0.1025" />
   <xacro:property name="link4_length" value="0.094" />
+  <xacro:property name="effector_length" value="0.05" />
   <xacro:property name="link1_d" value="-0.1405" />
   <xacro:property name="link2_d" value="0.1215" />
@@ -46,5 +47,5 @@
     <parent link="world"/>
     <child link="link0"/>
-    <origin xyz="${offset_x} ${offset_y} ${offset_z}" rpy="0 0 0"/>
+    <origin xyz="${offset_x} ${offset_y} ${offset_z}" rpy="0 0 ${-pi/2}"/>
     <axis xyz="0 0 1"/>
     <limit lower="${joint0_low}" upper="${joint0_high}" effort="${joint_effort_lim}" velocity="${joint_velocity_lim}"/>
@@ -328,5 +329,5 @@
     <parent link="link4" />
     <child link="effector" />
-    <origin xyz="0 0 ${link4_length + 0.05}" rpy="0 0 0" />
+    <origin xyz="0 0 ${link4_length + effector_length}" rpy="0 0 0" />
     <axis xyz="0 0 1" />
     <dynamics damping="0.5" />
@@ -335,19 +336,17 @@
   <link name="effector">
     <visual>
-      <origin xyz="0 0 0" rpy="0 0 0"/>
+      <origin xyz="0 0 0" rpy="0 0 0" />
       <geometry>
 	      <sphere radius="${marker_point_radius}" />
-        <!-- <mesh filename="$(find robot_sim)/mesh/cone.obj"
-              scale="0.4 0.4 0.5" /> -->
-      </geometry>
-      <material name="blue"/>
-    </visual>
-    <inertial>
-      <origin xyz="0 0 0" rpy="0 0 0"/>
-      <mass value="0.1"/>
-      <inertia
-        ixx="1.0" ixy="0.0" ixz="0.0"
-        iyy="1.0" iyz="0.0"
-        izz="1.0"/>
+      </geometry>
+      <material name="blue" />
+    </visual>
+    <inertial>
+      <origin xyz="0 0 0" rpy="0 0 0" />
+      <mass value="0.1" />
+      <inertia
+        ixx="1.0" ixy="0.0" ixz="0.0"
+        iyy="1.0" iyz="0.0"
+        izz="1.0" />
     </inertial>
   </link>

Commit message: desperate

File: src/RobotSimulator/src/robot_sim/urdf/markers.xacro (robot description, xacro)
@@ -5,4 +5,5 @@
   <!-- Base link -->
   <link name="world"/>
+  <!-- Red -->
   <joint name="marker_red_joint" type="fixed">
     <parent link="world"/>
@@ -29,3 +30,28 @@
     <material>Gazebo/Red</material>
   </gazebo>
+  <!-- Green -->
+  <joint name="marker_green_joint" type="fixed">
+    <parent link="world"/>
+    <child link="marker_green"/>
+  </joint>
+  <link name="marker_green">
+    <visual>
+      <origin xyz="0 0 0" rpy="0 0 0"/>
+      <geometry>
+	      <sphere radius="${marker_point_radius}" />
+      </geometry>
+      <material name="green"/>
+    </visual>
+    <inertial>
+      <origin xyz="0 0 0" rpy="0 0 0"/>
+      <mass value="1.0"/>
+      <inertia
+        ixx="1.0" ixy="0.0" ixz="0.0"
+        iyy="1.0" iyz="0.0"
+        izz="1.0"/>
+    </inertial>
+  </link>
+  <gazebo reference="marker_green">
+    <material>Gazebo/Green</material>
+  </gazebo>
 </robot>
