Commit message: Sync changes

File: src/RobotSimulator/src/robot_sim/urdf/robot.xacro (robot description, xacro)
@@ -17,4 +17,12 @@
   <xacro:property name="link2_length" value="0.5" />
   <xacro:property name="link3_length" value="0.4" />
+  <xacro:property name="joint1_low" value="0.0" />
+  <xacro:property name="joint1_high" value="${PI/2}" />
+  <xacro:property name="joint2_low" value="0.0" />
+  <xacro:property name="joint2_high" value="${PI/2}" />
+  <xacro:property name="joint3_low" value="0.0" />
+  <xacro:property name="joint3_high" value="${PI/2}" />
+  <xacro:property name="joint_effort_lim" value="2000" />
+  <xacro:property name="joint_velocity_lim" value="15" />
   <!-- Enable self-collision -->
   <gazebo>
@@ -101,10 +109,11 @@
   </gazebo>
   <!-- Joint 1 -->
-  <joint name="joint1" type="continuous">
+  <joint name="joint1" type="revolute">
     <parent link="link0" />
     <child link="link1" />
     <origin xyz="0 0 ${0.1 + link_gap/2}" rpy="0 0 0" />
     <axis xyz="0 1 0" />
-    <dynamics damping="0.7" />
+    <limit lower="${joint1_low}" upper="${joint1_high}" effort="${joint_effort_lim}" velocity="${joint_velocity_lim}"/>
+    <dynamics damping="0.5" />
   </joint>
   <transmission name="tran1">
@@ -159,10 +168,11 @@
   </gazebo>
   <!-- Joint 2 -->
-  <joint name="joint2" type="continuous">
+  <joint name="joint2" type="revolute">
     <parent link="link1" />
     <child link="link2" />
     <origin xyz="0 0 ${link1_length + link_gap}" rpy="0 0 0" />
     <axis xyz="0 1 0" />
-    <dynamics damping="0.7" />
+    <limit lower="${joint2_low}" upper="${joint2_high}" effort="${joint_effort_lim}" velocity="${joint_velocity_lim}"/>
+    <dynamics damping="0.5" />
   </joint>
   <transmission name="tran2">
@@ -217,10 +227,11 @@
   </gazebo>
   <!-- Joint 3 -->
-  <joint name="joint3" type="continuous">
+  <joint name="joint3" type="revolute">
     <parent link="link2" />
     <child link="link3" />
     <origin xyz="0 0 ${link2_length + link_gap}" rpy="0 0 0" />
     <axis xyz="0 1 0" />
-    <dynamics damping="0.7" />
+    <limit lower="${joint3_low}" upper="${joint3_high}" effort="${joint_effort_lim}" velocity="${joint_velocity_lim}"/>
+    <dynamics damping="0.5" />
   </joint>
   <transmission name="tran3">
@@ -280,5 +291,5 @@
     <origin xyz="0 0 ${link3_length + link_gap}" rpy="0 0 0" />
     <axis xyz="0 1 0" />
-    <dynamics damping="0.7" />
+    <dynamics damping="0.5" />
   </joint>
   <!-- Effector -->

Commit message: Sync changes

File: src/RobotSimulator/src/robot_sim/urdf/robot.xacro (robot description, xacro)
@@ -74,8 +74,8 @@
     <type>transmission_interface/SimpleTransmission</type>
     <joint name="joint0">
-      <hardwareInterface>hardware_interface/EffortJointInterface</hardwareInterface>
+      <hardwareInterface>hardware_interface/PositionJointInterface</hardwareInterface>
     </joint>
     <actuator name="motor0">
-      <hardwareInterface>hardware_interface/EffortJointInterface</hardwareInterface>
+      <hardwareInterface>hardware_interface/PositionJointInterface</hardwareInterface>
       <mechanicalReduction>1</mechanicalReduction>
     </actuator>
@@ -120,8 +120,8 @@
     <type>transmission_interface/SimpleTransmission</type>
     <joint name="joint1">
-      <hardwareInterface>hardware_interface/EffortJointInterface</hardwareInterface>
+      <hardwareInterface>hardware_interface/PositionJointInterface</hardwareInterface>
     </joint>
     <actuator name="motor1">
-      <hardwareInterface>hardware_interface/EffortJointInterface</hardwareInterface>
+      <hardwareInterface>hardware_interface/PositionJointInterface</hardwareInterface>
       <mechanicalReduction>1</mechanicalReduction>
     </actuator>
@@ -179,8 +179,8 @@
     <type>transmission_interface/SimpleTransmission</type>
     <joint name="joint2">
-      <hardwareInterface>hardware_interface/EffortJointInterface</hardwareInterface>
+      <hardwareInterface>hardware_interface/PositionJointInterface</hardwareInterface>
     </joint>
     <actuator name="motor2">
-      <hardwareInterface>hardware_interface/EffortJointInterface</hardwareInterface>
+      <hardwareInterface>hardware_interface/PositionJointInterface</hardwareInterface>
       <mechanicalReduction>1</mechanicalReduction>
     </actuator>
@@ -238,8 +238,8 @@
     <type>transmission_interface/SimpleTransmission</type>
     <joint name="joint3">
-      <hardwareInterface>hardware_interface/EffortJointInterface</hardwareInterface>
+      <hardwareInterface>hardware_interface/PositionJointInterface</hardwareInterface>
     </joint>
     <actuator name="motor3">
-      <hardwareInterface>hardware_interface/EffortJointInterface</hardwareInterface>
+      <hardwareInterface>hardware_interface/PositionJointInterface</hardwareInterface>
       <mechanicalReduction>1</mechanicalReduction>
     </actuator>

File: src/RobotSimulator/src/robot_sim/urdf/shared.xacro (robot description, xacro)
@@ -6,5 +6,5 @@
   <xacro:property name="PI" value="3.1415926535897931"/>
   <!-- Sensor parameters -->
-  <xacro:property name="sensor_update_rate" value="40.0"/>
+  <xacro:property name="sensor_update_rate" value="50.0"/>
   <!-- Marker parameters -->
   <xacro:property name="marker_point_radius" value="0.02"/>

Commit message: Sync changes

File: src/RobotSimulator/src/robot_sim/urdf/robot.xacro (robot description, xacro)
@@ -12,9 +12,15 @@
   </gazebo>
   <!-- Constants for robot dimensions -->
-  <xacro:property name="link_radius" value="0.05" />
-  <xacro:property name="link_gap" value="0.1" />
+  <xacro:property name="link_radius" value="0.04" />
+  <xacro:property name="offset_x" value="0" />
+  <xacro:property name="offset_y" value="0" />
+  <xacro:property name="offset_z" value="1" />
+  <xacro:property name="link0_length" value="0.2" />
   <xacro:property name="link1_length" value="0.5" />
   <xacro:property name="link2_length" value="0.5" />
-  <xacro:property name="link3_length" value="0.4" />
+  <xacro:property name="link3_length" value="0.3" />
+  <xacro:property name="link1_d" value="0.1" />
+  <xacro:property name="link2_d" value="-0.1" />
+  <xacro:property name="link3_d" value="0.1" />
   <xacro:property name="joint1_low" value="0.0" />
   <xacro:property name="joint1_high" value="${PI/2}" />
@@ -27,5 +33,5 @@
   <!-- Enable self-collision -->
   <gazebo>
-    <self_collide>true</self_collide>
+    <self_collide>false</self_collide>
   </gazebo>
   <!-- World link -->
@@ -35,5 +41,5 @@
     <parent link="world"/>
     <child link="link0"/>
-    <origin xyz="0 0 1.05" rpy="0 0 0"/>
+    <origin xyz="${offset_x} ${offset_y} ${offset_z}" rpy="0 0 0"/>
     <axis xyz="0 0 1"/>
     <dynamics damping="0.7"/>
@@ -52,18 +58,18 @@
   <link name="link0">
     <collision>
-      <origin xyz="0 0 0" rpy="0 0 0"/>
-      <geometry>
-	      <box size="0.5 0.5 0.1" />
-      </geometry>
-    </collision>
-    <visual>
-      <origin xyz="0 0 0" rpy="0 0 0"/>
-      <geometry>
-	      <box size="0.5 0.5 0.1" />
-      </geometry>
-      <material name="grey"/>
-    </visual>
-    <inertial>
-      <origin xyz="0 0 0" rpy="0 0 0" />
+      <origin xyz="0 0 ${link0_length/2}" rpy="0 0 0"/>
+      <geometry>
+	      <cylinder radius="${link_radius}" length="${link0_length}" />
+      </geometry>
+    </collision>
+    <visual>
+      <origin xyz="0 0 ${link0_length/2}" rpy="0 0 0"/>
+      <geometry>
+	      <cylinder radius="${link_radius}" length="${link0_length}" />
+      </geometry>
+      <material name="orange"/>
+    </visual>
+    <inertial>
+      <origin xyz="0 0 ${link0_length/2}" rpy="0 0 0" />
       <mass value="1.0"/>
       <inertia
@@ -74,5 +80,5 @@
   </link>
   <gazebo reference="link0">
-    <material>Gazebo/Grey</material>
+    <material>Gazebo/Orange</material>
   </gazebo>
   <!-- Joint 1 -->
@@ -80,5 +86,5 @@
     <parent link="link0" />
     <child link="link1" />
-    <origin xyz="0 0 ${0.1 + link_gap/2}" rpy="0 0 0" />
+    <origin xyz="0 ${link1_d} ${link0_length}" rpy="0 0 0" />
     <axis xyz="0 1 0" />
     <limit lower="${joint1_low}" upper="${joint1_high}" effort="${joint_effort_lim}" velocity="${joint_velocity_lim}"/>
@@ -98,5 +104,5 @@
   <link name="link1">
     <collision>
-      <origin xyz="0 0 ${link_gap/2 + link1_length/2}" rpy="0 0 0"/>
+      <origin xyz="0 0 ${link1_length/2}" rpy="0 0 0"/>
       <geometry>
 	      <cylinder radius="${link_radius}" length="${link1_length}" />
@@ -104,5 +110,5 @@
     </collision>
     <visual>
-      <origin xyz="0 0 ${link_gap/2 + link1_length/2}" rpy="0 0 0"/>
+      <origin xyz="0 0 ${link1_length/2}" rpy="0 0 0"/>
       <geometry>
 	      <cylinder radius="${link_radius}" length="${link1_length}" />
@@ -111,5 +117,5 @@
     </visual>
     <inertial>
-      <origin xyz="0 0 ${link_gap/2 + link1_length/2}" rpy="0 0 0"/>
+      <origin xyz="0 0 ${link1_length/2}" rpy="0 0 0"/>
       <mass value="1.0"/>
       <inertia
@@ -139,5 +145,5 @@
     <parent link="link1" />
     <child link="link2" />
-    <origin xyz="0 0 ${link1_length + link_gap}" rpy="0 0 0" />
+    <origin xyz="0 ${link2_d} ${link1_length}" rpy="0 0 0" />
     <axis xyz="0 1 0" />
     <limit lower="${joint2_low}" upper="${joint2_high}" effort="${joint_effort_lim}" velocity="${joint_velocity_lim}"/>
@@ -157,5 +163,5 @@
   <link name="link2">
     <collision>
-      <origin xyz="0 0 ${link_gap/2 + link2_length/2}" rpy="0 0 0"/>
+      <origin xyz="0 0 ${link2_length/2}" rpy="0 0 0"/>
       <geometry>
 	      <cylinder radius="${link_radius}" length="${link2_length}" />
@@ -163,5 +169,5 @@
     </collision>
     <visual>
-      <origin xyz="0 0 ${link_gap/2 + link2_length/2}" rpy="0 0 0"/>
+      <origin xyz="0 0 ${link2_length/2}" rpy="0 0 0"/>
       <geometry>
 	      <cylinder radius="${link_radius}" length="${link2_length}" />
@@ -170,5 +176,5 @@
     </visual>
     <inertial>
-      <origin xyz="0 0 ${link_gap/2 + link2_length/2}" rpy="0 0 0"/>
+      <origin xyz="0 0 ${link2_length/2}" rpy="0 0 0"/>
       <mass value="1.0"/>
       <inertia
@@ -198,5 +204,5 @@
     <parent link="link2" />
     <child link="link3" />
-    <origin xyz="0 0 ${link2_length + link_gap}" rpy="0 0 0" />
+    <origin xyz="0 ${link3_d} ${link2_length}" rpy="0 0 0" />
     <axis xyz="0 1 0" />
     <limit lower="${joint3_low}" upper="${joint3_high}" effort="${joint_effort_lim}" velocity="${joint_velocity_lim}"/>
@@ -216,5 +222,5 @@
   <link name="link3">
     <collision>
-      <origin xyz="0 0 ${link_gap/2 + link3_length/2}" rpy="0 0 0"/>
+      <origin xyz="0 0 ${link3_length/2}" rpy="0 0 0"/>
       <geometry>
 	      <cylinder radius="${link_radius}" length="${link3_length}" />
@@ -222,5 +228,5 @@
     </collision>
     <visual>
-      <origin xyz="0 0 ${link_gap/2 + link3_length/2}" rpy="0 0 0"/>
+      <origin xyz="0 0 ${link3_length/2}" rpy="0 0 0"/>
       <geometry>
 	      <cylinder radius="${link_radius}" length="${link3_length}" />
@@ -229,5 +235,5 @@
     </visual>
     <inertial>
-      <origin xyz="0 0 ${link_gap/2 + link3_length/2}" rpy="0 0 0"/>
+      <origin xyz="0 0 ${link3_length/2}" rpy="0 0 0"/>
       <mass value="1.0"/>
       <inertia
@@ -257,5 +263,5 @@
     <parent link="link3" />
     <child link="effector" />
-    <origin xyz="0 0 ${link3_length + link_gap}" rpy="0 0 0" />
+    <origin xyz="0 0 ${link3_length + 0.05}" rpy="0 0 0" />
     <axis xyz="0 1 0" />
     <dynamics damping="0.5" />

Commit message: Modify robot model

File: src/RobotSimulator/src/robot_sim/urdf/robot.xacro (robot description, xacro)
@@ -15,18 +15,23 @@
   <xacro:property name="offset_x" value="0" />
   <xacro:property name="offset_y" value="0" />
-  <xacro:property name="offset_z" value="1" />
-  <xacro:property name="link0_length" value="0.2" />
-  <xacro:property name="link1_length" value="0.5" />
-  <xacro:property name="link2_length" value="0.5" />
-  <xacro:property name="link3_length" value="0.3" />
-  <xacro:property name="link1_d" value="0.1" />
-  <xacro:property name="link2_d" value="-0.1" />
-  <xacro:property name="link3_d" value="0.1" />
-  <xacro:property name="joint1_low" value="0.0" />
-  <xacro:property name="joint1_high" value="${PI/2}" />
-  <xacro:property name="joint2_low" value="0.0" />
-  <xacro:property name="joint2_high" value="${PI/2}" />
-  <xacro:property name="joint3_low" value="0.0" />
-  <xacro:property name="joint3_high" value="${PI/2}" />
+  <xacro:property name="offset_z" value="0.2" />
+  <xacro:property name="link0_length" value="0.1215" />
+  <xacro:property name="link1_length" value="0.408" />
+  <xacro:property name="link2_length" value="0.376" />
+  <xacro:property name="link3_length" value="0.1025" />
+  <xacro:property name="link4_length" value="0.094" />
+  <xacro:property name="link1_d" value="-0.1405" />
+  <xacro:property name="link2_d" value="0.1215" />
+  <xacro:property name="link3_d" value="-0.1025" />
+  <xacro:property name="joint0_low" value="-0.000006" />
+  <xacro:property name="joint0_high" value="3.053448" />
+  <xacro:property name="joint1_low" value="-1.571984" />
+  <xacro:property name="joint1_high" value="1.571984" />
+  <xacro:property name="joint2_low" value="-1.529065" />
+  <xacro:property name="joint2_high" value="1.571069" />
+  <xacro:property name="joint3_low" value="-1.570796" />
+  <xacro:property name="joint3_high" value="1.570796" />
+  <xacro:property name="joint4_low" value="-3.053450" />
+  <xacro:property name="joint4_high" value="3.053439" />
   <xacro:property name="joint_effort_lim" value="2000" />
   <xacro:property name="joint_velocity_lim" value="15" />
@@ -38,9 +43,10 @@
   <link name="world"/>
   <!-- Joint 0 -->
-  <joint name="joint0" type="continuous">
+  <joint name="joint0" type="revolute">
     <parent link="world"/>
     <child link="link0"/>
     <origin xyz="${offset_x} ${offset_y} ${offset_z}" rpy="0 0 0"/>
     <axis xyz="0 0 1"/>
+    <limit lower="${joint0_low}" upper="${joint0_high}" effort="${joint_effort_lim}" velocity="${joint_velocity_lim}"/>
     <dynamics damping="0.7"/>
   </joint>
@@ -260,9 +266,68 @@
   </gazebo>
   <!-- Joint 4 -->
-  <joint name="joint4" type="continuous">
+  <joint name="joint4" type="revolute">
     <parent link="link3" />
+    <child link="link4" />
+    <origin xyz="0 0 ${link3_length}" rpy="${PI/2} 0 0" />
+    <axis xyz="0 1 0" />
+    <limit lower="${joint4_low}" upper="${joint4_high}" effort="${joint_effort_lim}" velocity="${joint_velocity_lim}"/>
+    <dynamics damping="0.5" />
+  </joint>
+  <transmission name="tran4">
+    <type>transmission_interface/SimpleTransmission</type>
+    <joint name="joint4">
+      <hardwareInterface>hardware_interface/PositionJointInterface</hardwareInterface>
+    </joint>
+    <actuator name="motor4">
+      <hardwareInterface>hardware_interface/PositionJointInterface</hardwareInterface>
+      <mechanicalReduction>1</mechanicalReduction>
+    </actuator>
+  </transmission>
+  <!-- Link 4 -->
+  <link name="link4">
+    <collision>
+      <origin xyz="0 0 ${link4_length/2}" rpy="0 0 0"/>
+      <geometry>
+	      <cylinder radius="${link_radius}" length="${link4_length}" />
+      </geometry>
+    </collision>
+    <visual>
+      <origin xyz="0 0 ${link4_length/2}" rpy="0 0 0"/>
+      <geometry>
+	      <cylinder radius="${link_radius}" length="${link4_length}" />
+      </geometry>
+      <material name="orange"/>
+    </visual>
+    <inertial>
+      <origin xyz="0 0 ${link4_length/2}" rpy="0 0 0"/>
+      <mass value="1.0"/>
+      <inertia
+        ixx="1.0" ixy="0.0" ixz="0.0"
+        iyy="1.0" iyz="0.0"
+        izz="1.0"/>
+    </inertial>
+  </link>
+  <gazebo reference="link4">
+    <material>Gazebo/Orange</material>
+  </gazebo>
+  <gazebo reference="link4">
+    <sensor name="link4_contact_sensor" type="contact">
+      <always_on>true</always_on>
+      <update_rate>${sensor_update_rate}</update_rate>
+      <visualize>false</visualize>
+      <contact>
+        <collision>link4_collision</collision>
+      </contact>
+      <plugin name="gazebo_ros_bumper_controller" filename="libgazebo_ros_bumper.so">
+        <bumperTopicName>/link4_bumper</bumperTopicName>
+      </plugin>
+    </sensor>
+  </gazebo>
+  <!-- Joint 5 -->
+  <joint name="joint5" type="continuous">
+    <parent link="link4" />
     <child link="effector" />
-    <origin xyz="0 0 ${link3_length + 0.05}" rpy="0 0 0" />
-    <axis xyz="0 1 0" />
+    <origin xyz="0 0 ${link4_length + 0.05}" rpy="0 0 0" />
+    <axis xyz="0 0 1" />
     <dynamics damping="0.5" />
   </joint>
@@ -273,4 +338,6 @@
       <geometry>
 	      <sphere radius="${marker_point_radius}" />
+        <!-- <mesh filename="$(find robot_sim)/mesh/cone.obj"
+              scale="0.4 0.4 0.5" /> -->
       </geometry>
       <material name="blue"/>

Commit message: Optimize A*

File: src/RobotSimulator/src/robot_sim/urdf/robot.xacro (robot description, xacro)
@@ -64,10 +64,10 @@
   <!-- Link 0 -->
   <link name="link0">
-    <collision>
+    <!-- <collision>
       <origin xyz="0 0 ${link0_length/2}" rpy="0 0 0"/>
       <geometry>
 	      <cylinder radius="${link_radius}" length="${link0_length}" />
       </geometry>
-    </collision>
+    </collision> -->
     <visual>
       <origin xyz="0 0 ${link0_length/2}" rpy="0 0 0"/>
