Commit message: Sync changes (incomplete)

File: src/RobotSimulator/src/robot_sim/urdf/obstacles.xacro (robot description, xacro)
@@ -1,13 +1,6 @@
 <?xml version="1.0"?>
-<robot name="obstacle" xmlns:xacro="http://www.ros.org/wiki/xacro">
+<robot name="obstacles" xmlns:xacro="http://www.ros.org/wiki/xacro">
   <!-- Import shared components -->
   <xacro:include filename="$(find robot_sim)/urdf/shared.xacro" />
-  <!-- ros_control plugin -->
-  <gazebo>
-    <plugin name="gazebo_ros_control" filename="libgazebo_ros_control.so">
-      <robotNamespace>/obstacle</robotNamespace>
-      <robotSimType>gazebo_ros_control/DefaultRobotHWSim</robotSimType>
-    </plugin>
-  </gazebo>
   <!-- Base link -->
   <link name="world"/>

File: src/RobotSimulator/src/robot_sim/urdf/robot.xacro (robot description, xacro)
@@ -148,5 +148,5 @@
     <sensor name="link1_contact_sensor" type="contact">
       <always_on>true</always_on>
-      <update_rate>20.0</update_rate>
+      <update_rate>${sensor_update_rate}</update_rate>
       <visualize>false</visualize>
       <contact>
@@ -206,5 +206,5 @@
     <sensor name="link2_contact_sensor" type="contact">
       <always_on>true</always_on>
-      <update_rate>20.0</update_rate>
+      <update_rate>${sensor_update_rate}</update_rate>
       <visualize>false</visualize>
       <contact>
@@ -264,5 +264,5 @@
     <sensor name="link3_contact_sensor" type="contact">
       <always_on>true</always_on>
-      <update_rate>20.0</update_rate>
+      <update_rate>${sensor_update_rate}</update_rate>
       <visualize>false</visualize>
       <contact>
@@ -274,3 +274,32 @@
     </sensor>
   </gazebo>
+  <!-- Joint 4 -->
+  <joint name="joint4" type="continuous">
+    <parent link="link3" />
+    <child link="effector" />
+    <origin xyz="0 0 ${link3_length + link_gap}" rpy="0 0 0" />
+    <axis xyz="0 1 0" />
+    <dynamics damping="0.7" />
+  </joint>
+  <!-- Effector -->
+  <link name="effector">
+    <visual>
+      <origin xyz="0 0 0" rpy="0 0 0"/>
+      <geometry>
+	      <sphere radius="${marker_point_radius}" />
+      </geometry>
+      <material name="blue"/>
+    </visual>
+    <inertial>
+      <origin xyz="0 0 0" rpy="0 0 0"/>
+      <mass value="0.1"/>
+      <inertia
+        ixx="1.0" ixy="0.0" ixz="0.0"
+        iyy="1.0" iyz="0.0"
+        izz="1.0"/>
+    </inertial>
+  </link>
+  <gazebo reference="effector">
+    <material>Gazebo/Blue</material>
+  </gazebo>
 </robot>

File: src/RobotSimulator/src/robot_sim/urdf/shared.xacro (robot description, xacro)
@@ -1,7 +1,11 @@
 <?xml version="1.0"?>
 <robot xmlns:xacro="http://www.ros.org/wiki/xacro">
-  <!-- Import constants -->
-  <xacro:property name="PI" value="3.1415926535897931"/>
   <!-- Import Rviz colors -->
   <xacro:include filename="$(find robot_sim)/urdf/materials.xacro" />
+  <!-- Math constants -->
+  <xacro:property name="PI" value="3.1415926535897931"/>
+  <!-- Sensor parameters -->
+  <xacro:property name="sensor_update_rate" value="40.0"/>
+  <!-- Marker parameters -->
+  <xacro:property name="marker_point_radius" value="0.02"/>
 </robot>

Commit message: Sync changes (incomplete)

File: src/RobotSimulator/src/robot_sim/urdf/obstacles.xacro (robot description, xacro)
@@ -5,4 +5,37 @@
   <!-- Base link -->
   <link name="world"/>
+  <!-- Table -->
+  <joint name="joint_table" type="fixed">
+    <parent link="world"/>
+    <child link="table"/>
+    <origin xyz="0 0 0.5" rpy="0 0 0"/>
+  </joint>
+  <link name="table">
+    <collision>
+      <origin xyz="0 0 0" rpy="0 0 0"/>
+      <geometry>
+	      <box size="1 1 1" />
+      </geometry>
+    </collision>
+    <visual>
+      <origin xyz="0 0 0" rpy="0 0 0"/>
+      <geometry>
+	      <box size="1 1 1" />
+      </geometry>
+      <material name="white"/>
+    </visual>
+    <inertial>
+      <origin xyz="0 0 0" rpy="0 0 0"/>
+      <mass value="1.0"/>
+      <inertia
+        ixx="1.0" ixy="0.0" ixz="0.0"
+        iyy="1.0" iyz="0.0"
+        izz="1.0"/>
+    </inertial>
+  </link>
+  <gazebo reference="table">
+    <material>Gazebo/White</material>
+  </gazebo>
+  <!-- Obj 1 -->
   <joint name="obj1_joint" type="fixed">
     <parent link="world"/>
@@ -11,18 +44,18 @@
   <link name="obj1">
     <collision>
-      <origin xyz="0.5 0 2" rpy="0 0 0"/>
+      <origin xyz="0.701 0.701 2" rpy="0 0 0"/>
       <geometry>
-	      <box size="0.5 0.5 0.5"/>
+	      <box size="0.302 0.302 4"/>
       </geometry>
     </collision>
     <visual>
-      <origin xyz="0.5 0 2" rpy="0 0 0"/>
+      <origin xyz="0.701 0.701 2" rpy="0 0 0"/>
       <geometry>
-	      <box size="0.5 0.5 0.5"/>
+	      <box size="0.302 0.302 4"/>
       </geometry>
-      <material name="blue"/>
+      <material name="white"/>
     </visual>
     <inertial>
-      <origin xyz="0.5 0 2" rpy="0 0 0"/>
+      <origin xyz="0.701 0.701 2" rpy="0 0 0"/>
       <mass value="1.0"/>
       <inertia
@@ -33,5 +66,98 @@
   </link>
   <gazebo reference="obj1">
-    <material>Gazebo/Blue</material>
+    <material>Gazebo/White</material>
+  </gazebo>
+  <!-- Obj 2 -->
+  <joint name="obj2_joint" type="fixed">
+    <parent link="world"/>
+    <child link="obj2"/>
+  </joint>
+  <link name="obj2">
+    <collision>
+      <origin xyz="0.701 -0.701 2" rpy="0 0 0"/>
+      <geometry>
+	      <box size="0.302 0.302 4"/>
+      </geometry>
+    </collision>
+    <visual>
+      <origin xyz="0.701 -0.701 2" rpy="0 0 0"/>
+      <geometry>
+	      <box size="0.302 0.302 4"/>
+      </geometry>
+      <material name="white"/>
+    </visual>
+    <inertial>
+      <origin xyz="0.701 -0.701 2" rpy="0 0 0"/>
+      <mass value="1.0"/>
+      <inertia
+        ixx="1.0" ixy="0.0" ixz="0.0"
+        iyy="1.0" iyz="0.0"
+        izz="1.0"/>
+    </inertial>
+  </link>
+  <gazebo reference="obj2">
+    <material>Gazebo/White</material>
+  </gazebo>
+  <!-- Obj 3 -->
+  <joint name="obj3_joint" type="fixed">
+    <parent link="world"/>
+    <child link="obj3"/>
+  </joint>
+  <link name="obj3">
+    <collision>
+      <origin xyz="-0.701 0.701 2" rpy="0 0 0"/>
+      <geometry>
+	      <box size="0.302 0.302 4"/>
+      </geometry>
+    </collision>
+    <visual>
+      <origin xyz="-0.701 0.701 2" rpy="0 0 0"/>
+      <geometry>
+	      <box size="0.302 0.302 4"/>
+      </geometry>
+      <material name="white"/>
+    </visual>
+    <inertial>
+      <origin xyz="-0.701 0.701 2" rpy="0 0 0"/>
+      <mass value="1.0"/>
+      <inertia
+        ixx="1.0" ixy="0.0" ixz="0.0"
+        iyy="1.0" iyz="0.0"
+        izz="1.0"/>
+    </inertial>
+  </link>
+  <gazebo reference="obj3">
+    <material>Gazebo/White</material>
+  </gazebo>
+  <!-- Obj 4 -->
+  <joint name="obj4_joint" type="fixed">
+    <parent link="world"/>
+    <child link="obj4"/>
+  </joint>
+  <link name="obj4">
+    <collision>
+      <origin xyz="-0.701 -0.701 2" rpy="0 0 0"/>
+      <geometry>
+	      <box size="0.302 0.302 4"/>
+      </geometry>
+    </collision>
+    <visual>
+      <origin xyz="-0.701 -0.701 2" rpy="0 0 0"/>
+      <geometry>
+	      <box size="0.302 0.302 4"/>
+      </geometry>
+      <material name="white"/>
+    </visual>
+    <inertial>
+      <origin xyz="-0.701 -0.701 2" rpy="0 0 0"/>
+      <mass value="1.0"/>
+      <inertia
+        ixx="1.0" ixy="0.0" ixz="0.0"
+        iyy="1.0" iyz="0.0"
+        izz="1.0"/>
+    </inertial>
+  </link>
+  <gazebo reference="obj4">
+    <material>Gazebo/White</material>
   </gazebo>
 </robot>

File: src/RobotSimulator/src/robot_sim/urdf/robot.xacro (robot description, xacro)
@@ -31,41 +31,9 @@
   <!-- World link -->
   <link name="world"/>
-  <!-- Table -->
-  <joint name="joint_table" type="fixed">
-    <parent link="world"/>
-    <child link="table"/>
-    <origin xyz="0 0 0.5" rpy="0 0 0"/>
-  </joint>
-  <link name="table">
-    <collision>
-      <origin xyz="0 0 0" rpy="0 0 0"/>
-      <geometry>
-	      <box size="1 1 1" />
-      </geometry>
-    </collision>
-    <visual>
-      <origin xyz="0 0 0" rpy="0 0 0"/>
-      <geometry>
-	      <box size="1 1 1" />
-      </geometry>
-      <material name="white"/>
-    </visual>
-    <inertial>
-      <origin xyz="0 0 0" rpy="0 0 0"/>
-      <mass value="1.0"/>
-      <inertia
-        ixx="1.0" ixy="0.0" ixz="0.0"
-        iyy="1.0" iyz="0.0"
-        izz="1.0"/>
-    </inertial>
-  </link>
-  <gazebo reference="table">
-    <material>Gazebo/White</material>
-  </gazebo>
   <!-- Joint 0 -->
   <joint name="joint0" type="continuous">
-    <parent link="table"/>
+    <parent link="world"/>
     <child link="link0"/>
-    <origin xyz="0 0 0.55" rpy="0 0 0"/>
+    <origin xyz="0 0 1.05" rpy="0 0 0"/>
     <axis xyz="0 0 1"/>
     <dynamics damping="0.7"/>

Commit message: Test RL (simple reward)

File: src/RobotSimulator/src/robot_sim/urdf/obstacles.xacro (robot description, xacro)
@@ -15,5 +15,5 @@
       <origin xyz="0 0 0" rpy="0 0 0"/>
       <geometry>
-	      <box size="1 1 0.2" />
+	      <box size="1 1 0.19" />
       </geometry>
     </collision>
@@ -21,5 +21,5 @@
       <origin xyz="0 0 0" rpy="0 0 0"/>
       <geometry>
-	      <box size="1 1 0.2" />
+	      <box size="1 1 0.19" />
       </geometry>
       <material name="white"/>

Commit message: Sync changes

File: src/RobotSimulator/src/robot_sim/urdf/obstacles.xacro (robot description, xacro)
@@ -165,3 +165,131 @@
     <material>Gazebo/White</material>
   </gazebo>
+  <!-- Obj 5 -->
+  <!-- <joint name="obj5_joint" type="fixed">
+    <parent link="world"/>
+    <child link="obj5"/>
+    <origin xyz="0.3 0.3 0.8" rpy="0 0 0"/>
+  </joint>
+  <link name="obj5">
+    <collision>
+      <origin xyz="0 0 0" rpy="0 0 0"/>
+      <geometry>
+	      <box size="0.15 0.15 0.15"/>
+      </geometry>
+    </collision>
+    <visual>
+      <origin xyz="0 0 0" rpy="0 0 0"/>
+      <geometry>
+	      <box size="0.15 0.15 0.15"/>
+      </geometry>
+      <material name="white"/>
+    </visual>
+    <inertial>
+      <origin xyz="0 0 0" rpy="0 0 0"/>
+      <mass value="1.0"/>
+      <inertia
+        ixx="1.0" ixy="0.0" ixz="0.0"
+        iyy="1.0" iyz="0.0"
+        izz="1.0"/>
+    </inertial>
+  </link>
+  <gazebo reference="obj5">
+    <material>Gazebo/White</material>
+  </gazebo> -->
+  <!-- Obj 6 -->
+  <!-- <joint name="obj6_joint" type="fixed">
+    <parent link="world"/>
+    <child link="obj6"/>
+    <origin xyz="0.3 -0.3 0.8" rpy="0 0 0"/>
+  </joint>
+  <link name="obj6">
+    <collision>
+      <origin xyz="0 0 0" rpy="0 0 0"/>
+      <geometry>
+	      <box size="0.15 0.15 0.15"/>
+      </geometry>
+    </collision>
+    <visual>
+      <origin xyz="0 0 0" rpy="0 0 0"/>
+      <geometry>
+	      <box size="0.15 0.15 0.15"/>
+      </geometry>
+      <material name="white"/>
+    </visual>
+    <inertial>
+      <origin xyz="0 0 0" rpy="0 0 0"/>
+      <mass value="1.0"/>
+      <inertia
+        ixx="1.0" ixy="0.0" ixz="0.0"
+        iyy="1.0" iyz="0.0"
+        izz="1.0"/>
+    </inertial>
+  </link>
+  <gazebo reference="obj6">
+    <material>Gazebo/White</material>
+  </gazebo> -->
+  <!-- Obj 7 -->
+  <!-- <joint name="obj7_joint" type="fixed">
+    <parent link="world"/>
+    <child link="obj7"/>
+    <origin xyz="-0.3 0.3 0.8" rpy="0 0 0"/>
+  </joint>
+  <link name="obj7">
+    <collision>
+      <origin xyz="0 0 0" rpy="0 0 0"/>
+      <geometry>
+	      <box size="0.15 0.15 0.15"/>
+      </geometry>
+    </collision>
+    <visual>
+      <origin xyz="0 0 0" rpy="0 0 0"/>
+      <geometry>
+	      <box size="0.15 0.15 0.15"/>
+      </geometry>
+      <material name="white"/>
+    </visual>
+    <inertial>
+      <origin xyz="0 0 0" rpy="0 0 0"/>
+      <mass value="1.0"/>
+      <inertia
+        ixx="1.0" ixy="0.0" ixz="0.0"
+        iyy="1.0" iyz="0.0"
+        izz="1.0"/>
+    </inertial>
+  </link>
+  <gazebo reference="obj7">
+    <material>Gazebo/White</material>
+  </gazebo> -->
+  <!-- Obj 8 -->
+  <!-- <joint name="obj8_joint" type="fixed">
+    <parent link="world"/>
+    <child link="obj8"/>
+    <origin xyz="-0.3 -0.3 0.8" rpy="0 0 0"/>
+  </joint>
+  <link name="obj8">
+    <collision>
+      <origin xyz="0 0 0" rpy="0 0 0"/>
+      <geometry>
+	      <box size="0.15 0.15 0.15"/>
+      </geometry>
+    </collision>
+    <visual>
+      <origin xyz="0 0 0" rpy="0 0 0"/>
+      <geometry>
+	      <box size="0.15 0.15 0.15"/>
+      </geometry>
+      <material name="white"/>
+    </visual>
+    <inertial>
+      <origin xyz="0 0 0" rpy="0 0 0"/>
+      <mass value="1.0"/>
+      <inertia
+        ixx="1.0" ixy="0.0" ixz="0.0"
+        iyy="1.0" iyz="0.0"
+        izz="1.0"/>
+    </inertial>
+  </link>
+  <gazebo reference="obj8">
+    <material>Gazebo/White</material>
+  </gazebo> -->
 </robot>
